File: tm-pulses.kicad_pcb (KiCad board)
At the start: 2 copper layers, 30 x 241 mm, 72 parts, among them J1 Conn_02x08_Odd_Even, J10 OUT24, J11 OUT47, J12 OUT1247, J2 OUT1, J3 OUT2, J4 OUT3, J5 OUT4, J6 OUT5, J7 OUT6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

Commit message: prefab checklist v0
Other:
- board text added: "PULSES (from TURING MACHINE) <---"
Changed lines of the file:
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@@
     )
   )
+  (gr_line (start 130.048 133.604) (end 129.032 132.588)
+    (stroke (width 0.15) (type default)) (layer "F.SilkS"))
+  (gr_line (start 144.018 141.732) (end 143.002 140.716)
+    (stroke (width 0.15) (type default)) (layer "F.SilkS"))
+  (gr_line (start 144.018 126.238) (end 144.018 125.73)
+    (stroke (width 0.15) (type default)) (layer "F.SilkS"))
+  (gr_line (start 130.048 180.848) (end 129.032 179.832)
+    (stroke (width 0.15) (type default)) (layer "F.SilkS"))
+  (gr_line (start 130.048 197.104) (end 130.048 196.596)
+    (stroke (width 0.15) (type default)) (layer "F.SilkS"))
+  (gr_line (start 144.018 204.216) (end 143.002 203.2)
+    (stroke (width 0.15) (type default)) (layer "F.SilkS"))
+  (gr_line (start 130.048 165.608) (end 130.048 165.1)
+    (stroke (width 0.15) (type default)) (layer "F.SilkS"))
+  (gr_line (start 130.048 149.352) (end 129.032 148.336)
+    (stroke (width 0.15) (type default)) (layer "F.SilkS"))
+  (gr_line (start 130.048 149.86) (end 130.048 149.352)
+    (stroke (width 0.15) (type default)) (layer "F.SilkS"))
+  (gr_line (start 130.048 134.112) (end 130.048 133.604)
+    (stroke (width 0.15) (type default)) (layer "F.SilkS"))
+  (gr_line (start 130.048 165.1) (end 129.032 164.084)
+    (stroke (width 0.15) (type default)) (layer "F.SilkS"))
+  (gr_line (start 144.018 188.468) (end 143.002 187.452)
+    (stroke (width 0.15) (type default)) (layer "F.SilkS"))
+  (gr_line (start 130.048 196.596) (end 129.032 195.58)
+    (stroke (width 0.15) (type default)) (layer "F.SilkS"))
+  (gr_line (start 144.018 142.24) (end 144.018 141.732)
+    (stroke (width 0.15) (type default)) (layer "F.SilkS"))
+  (gr_line (start 130.048 212.852) (end 130.048 212.344)
+    (stroke (width 0.15) (type default)) (layer "F.SilkS"))
+  (gr_line (start 130.048 117.856) (end 129.032 116.84)
+    (stroke (width 0.15) (type default)) (layer "F.SilkS"))
+  (gr_line (start 130.048 181.356) (end 130.048 180.848)
+    (stroke (width 0.15) (type default)) (layer "F.SilkS"))
+  (gr_line (start 144.018 204.724) (end 144.018 204.216)
+    (stroke (width 0.15) (type default)) (layer "F.SilkS"))
+  (gr_line (start 130.048 118.364) (end 130.048 117.856)
+    (stroke (width 0.15) (type default)) (layer "F.SilkS"))
+  (gr_line (start 144.018 188.976) (end 144.018 188.468)
+    (stroke (width 0.15) (type default)) (layer "F.SilkS"))
+  (gr_line (start 130.048 212.344) (end 129.032 211.328)
+    (stroke (width 0.15) (type default)) (layer "F.SilkS"))
+  (gr_line (start 144.018 125.73) (end 143.002 124.714)
+    (stroke (width 0.15) (type default)) (layer "F.SilkS"))
   (gr_rect (start 122.16 -8.4) (end 152.16 101.6)
     (stroke (width 0.1) (type default)) (fill none) (layer "Edge.Cuts"))
@@
     (effects (font (size 1 1) (thickness 0.15)) (justify left bottom mirror))
   )
+  (gr_text "PULSES\n(from TURING MACHINE)\n<---" (at 142.24 40.894) (layer "B.SilkS")
+    (effects (font (size 1 1) (thickness 0.15)) (justify left bottom mirror))
+  )
